Commit message: Its kind of working, need to have more power or less dynamics

File: robot/snake_robot.urdf (robot description, URDF)
Before this commit: robot snake_robot, 10 links, 9 joints
Links:
- link base_link: mass 1.0 -> 1000.0
Joints:
- joint joint8: axis 1 0 0 -> 0 1 0

Commit message: working

File: robot/snake_robot.urdf (robot description, URDF)
Before this commit: robot snake_robot, 10 links, 9 joints
Links:
- added link link11, mass 1.0; collision box size=0.1 0.1 0.5; visual box size=0.1 0.1 0.5
- added link link12, mass 1.0; collision box size=0.1 0.1 0.5; visual box size=0.1 0.1 0.5
- added link link13, mass 1.0; collision box size=0.1 0.1 0.5; visual box size=0.1 0.1 0.5
- added link link14, mass 1.0; collision box size=0.1 0.1 0.5; visual box size=0.1 0.1 0.5
- added link link15, mass 1.0; collision box size=0.1 0.1 0.5; visual box size=0.1 0.1 0.5
- added link link16, mass 1.0; collision box size=0.1 0.1 0.5; visual box size=0.1 0.1 0.5
- link base_link: mass 1000.0 -> 1.0; geometry collision box size=0.1 0.1 0.5; visual box size=0.1 0.1 0.5
- link link10: geometry collision box size=0.1 0.1 0.5; visual box size=0.1 0.1 0.5
- link link2: geometry collision box size=0.1 0.1 0.5; visual box size=0.1 0.1 0.5
- link link3: geometry collision box size=0.1 0.1 0.5; visual box size=0.1 0.1 0.5
- link link4: geometry collision box size=0.1 0.1 0.5; visual box size=0.1 0.1 0.5
- link link5: geometry collision box size=0.1 0.1 0.5; visual box size=0.1 0.1 0.5
- link link6: geometry collision box size=0.1 0.1 0.5; visual box size=0.1 0.1 0.5
- link link7: geometry collision box size=0.1 0.1 0.5; visual box size=0.1 0.1 0.5
- link link8: geometry collision box size=0.1 0.1 0.5; visual box size=0.1 0.1 0.5
- link link9: geometry collision box size=0.1 0.1 0.5; visual box size=0.1 0.1 0.5
Joints:
- added joint joint10: type continuous, parent link10, child link11, origin xyz= 0 0 0.5 rpy=0 0 0, axis 0 1 0
- added joint joint11: type continuous, parent link11, child link12, origin xyz= 0 0 0.5 rpy=0 0 0, axis 1 0 0
- added joint joint12: type continuous, parent link12, child link13, origin xyz= 0 0 0.5 rpy=0 0 0, axis 0 1 0
- added joint joint13: type continuous, parent link13, child link14, origin xyz= 0 0 0.5 rpy=0 0 0, axis 1 0 0
- added joint joint14: type continuous, parent link14, child link15, origin xyz= 0 0 0.5 rpy=0 0 0, axis 0 1 0
- added joint joint15: type continuous, parent link15, child link16, origin xyz= 0 0 0.5 rpy=0 0 0, axis 1 0 0
